File: vga/vga_sync.kicad_pcb (KiCad board)
At the start: 4 copper layers, 129.8 x 78.7 mm, 58 parts, among them J1 Conn_01x40, U1 74AC163, U10 74AC112, U11 74AC74, U12 74AC163, U13 74AC163, U14 74AC163, U16 74AC574, U17 74AC574, U18 74AC574, U19 74AC574, U2 74AC163, U3 74AC163, U4 74AC20, U5 74AC20, U6 74AC04, U7 74AC11, U8 74AC10, U9 74AC74, X1 25.175Mhz

Commit message: Update vga
Parts:
- added JP1: VSYNC, Jumper:SolderJumper-3_P1.3mm_Open_RoundedPad1.0x1.5mm, B.Cu at (229.8, 80.2)
- added JP2: HSYNC, Jumper:SolderJumper-3_P1.3mm_Open_RoundedPad1.0x1.5mm, B.Cu at (223.4, 80.2)
- added JP3: DISPLAY, Jumper:SolderJumper-3_P1.3mm_Open_RoundedPad1.0x1.5mm, B.Cu at (217.1, 80.2)
Connections:
- U18 pad 6: Net-(U18-Pad6) -> VCC
- U18 pad 7: Net-(U18-Pad7) -> VCC
- U18 pad 8: Net-(U18-Pad8) -> VCC
- U18 pad 9: Net-(U18-Pad9) -> VCC
- U19 pad 15: Net-(J1-Pad40) -> Net-(JP1-Pad3)
- U19 pad 16: Net-(J1-Pad38) -> Net-(JP2-Pad3)
- U19 pad 17: Net-(J1-Pad37) -> Net-(JP3-Pad3)
- U19 pad 7: Net-(U19-Pad7) -> Net-(JP3-Pad3)
- U19 pad 8: Net-(U19-Pad8) -> Net-(JP2-Pad3)
- U19 pad 9: Net-(U19-Pad9) -> Net-(JP1-Pad3)
Routing:
- net Net-(JP1-Pad3): track 0.00 -> 20.9 mm
- net Net-(JP2-Pad3): track 0.00 -> 17.0 mm
- net Net-(JP3-Pad3): track 0.00 -> 15.4 mm
- net Net-(J1-Pad40): track 33.4 -> 41.6 mm
- net Net-(JP3-Pad1): track 0.00 -> 7.31 mm, vias 0 -> 1
- net Net-(JP1-Pad1): track 0.00 -> 5.66 mm
- net Net-(J1-Pad38): track 33.4 -> 38.0 mm
- net Net-(JP2-Pad1): track 0.00 -> 4.49 mm, vias 0 -> 1
- net Net-(J1-Pad37): track 29.8 -> 30.7 mm
- net VCC: vias 53 -> 63
- net GND: vias 72 -> 67
