File: 7segment/7segment.kicad_sch (KiCad schematic)
At the start: 30 parts, among them J1 AVR-ISP-6, J2 Conn_01x10, J4 Conn_01x02, Q1 Q_NPN_BEC, Q2 Q_NPN_BEC, U1 ATmega168PA-AU, U2 HDSP-523

Commit message: Update
Other:
- note added: "At 50% duty cycle: Red 270 ohms Green 120 ohms Yellow 100 ohms"
Changed lines of the file:
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@@
     (stroke (width 0) (type default) (color 0 0 0 0))
+  )
+  (text "At 50% duty cycle:\nRed    270 ohms\nGreen  120 ohms\nYellow 100 ohms"
+    (at 243.84 77.47 0)
+    (effects (font (size 1.27 1.27)) (justify left bottom))
   )
   (label "DIG_F" (at 236.22 74.93 180)
